File: flipflop_beginners/flipflop/flipflop.kicad_pcb (KiCad board)
At the start: 2 copper layers, 100 x 50 mm, 10 parts, among them SW1 ON, SW2 OFF, U1 CD40107BE

Commit message: flipflop pcb redesign
Parts:
- moved D1 35.0 mm to (90.0, 21.0)
- moved R5 35.0 mm to (101.2, 21.0)
- moved SW2 30.2 mm to (19.8, 53.8)
- moved SW1 25.3 mm to (101.0, 54.0)
- moved R3 21.1 mm to (60.0, 19.2)
- moved R4 17.7 mm to (68.0, 19.2)
- moved R2 13.4 mm to (26.0, 30.0), turned to -90 degrees
- moved R1 10.5 mm to (101.0, 30.2), turned to -90 degrees
- moved U1 3.61 mm to (60.2, 34.2)
Routing:
- net +9V: track 84.8 -> 109.7 mm
- net /Off_Button: track 34.3 -> 58.4 mm
- net /On_Button: track 41.7 -> 56.3 mm
- net Net-(D1-Pad2): track 40.1 -> 44.8 mm
- net Net-(R3-Pad2): track 17.7 -> 21.1 mm
