File: blinker_beginners/blinker/blinker.kicad_pcb (KiCad board)
At the start: 2 copper layers, 100 x 50 mm, 7 parts, among them U1 NE555P

Commit message: Hold Enable Button for Blink
Parts:
- added SW1: SW_MEC_5E, switch_footprints:SW_PUSH_6mm, F.Cu at (37.0, 28.0)
Connections:
- BT1 pad 1: +9V -> Net-(BT1-Pad1)
Routing:
- net Net-(BT1-Pad1): track 0.00 -> 13.4 mm
Changed lines of the file:
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@@
   (net 6 "/Discharge")
   (net 7 "unconnected-(U1-Pad5)")
+  (net 8 "Net-(BT1-Pad1)")
   (footprint "Connector_PinHeader_2.54mm:PinHeader_1x02_P2.54mm_Vertical" (layer "F.Cu")
     (at 28 25 -90)
@@
     (fp_line (start -0.635 -1.27) (end 1.27 -1.27) (layer "F.Fab") (width 0.1))
     (pad "1" thru_hole rect (at 0 0 270) (size 1.7 1.7) (drill 1) (layers *.Cu *.Mask)
-      (net 1 "+9V") (pinfunction "+") (pintype "passive"))
+      (net 8 "Net-(BT1-Pad1)") (pinfunction "+") (pintype "passive"))
     (pad "2" thru_hole oval (at 0 2.54 270) (size 1.7 1.7) (drill 1) (layers *.Cu *.Mask)
       (net 2 "GND") (pinfunction "-") (pintype "passive"))
@@
     )
   )
+  (footprint "switch_footprints:SW_PUSH_6mm" (layer "F.Cu")
+    (at 37 28 -90)
+    (descr "https://www.omron.com/ecb/products/pdf/en-b3f.pdf")
+    (tags "tact sw push 6mm")
+    (property "Sheetfile" "blinker.kicad_sch")
+    (property "Sheetname" "")
+    (attr through_hole)
+    (fp_text reference "SW1" (at 0 -4.25 90) (layer "F.SilkS")
+      (effects (font (size 1 1) (thickness 0.15)))
+    )
+    (fp_text value "SW_MEC_5E" (at 0.5 4.45 90) (layer "F.Fab")
+      (effects (font (size 1 1) (thickness 0.15)))
+    )
+    (fp_text user "${REFERENCE}" (at 0 0 90) (layer "F.Fab")
+      (effects (font (size 1 1) (thickness 0.15)))
+    )
+    (fp_line (start -3.5 -0.75) (end -3.5 0.75) (layer "F.SilkS") (width 0.12))
+    (fp_line (start 3.5 0.75) (end 3.5 -0.75) (layer "F.SilkS") (width 0.12))
+    (fp_line (start 2.25 -3.25) (end -2.25 -3.25) (layer "F.SilkS") (width 0.12))
+    (fp_line (start -2.25 3.25) (end 2.25 3.25) (layer "F.SilkS") (width 0.12))
+    (fp_line (start -4.5 -3.75) (end 4.5 -3.75) (layer "F.CrtYd") (width 0.05))
+    (fp_line (start 4.75 -3.75) (end 4.75 -3.5) (layer "F.CrtYd") (width 0.05))
+    (fp_line (start 4.5 3.75) (end -4.5 3.75) (layer "F.CrtYd") (width 0.05))
+    (fp_line (start 4.5 -3.75) (end 4.75 -3.75) (layer "F.CrtYd") (width 0.05))
+    (fp_line (start -4.75 3.5) (end -4.75 -3.5) (layer "F.CrtYd") (width 0.05))
+    (fp_line (start 4.75 3.75) (end 4.75 3.5) (layer "F.CrtYd") (width 0.05))
+    (fp_line (start -4.75 -3.75) (end -4.5 -3.75) (layer "F.CrtYd") (width 0.05))
+    (fp_line (start -4.75 3.5) (end -4.75 3.75) (layer "F.CrtYd") (width 0.05))
+    (fp_line (start 4.75 -3.5) (end 4.75 3.5) (layer "F.CrtYd") (width 0.05))
+    (fp_line (start -4.75 -3.5) (end -4.75 -3.75) (layer "F.CrtYd") (width 0.05))
+    (fp_line (start -4.75 3.75) (end -4.5 3.75) (layer "F.CrtYd") (width 0.05))
+    (fp_line (start 4.5 3.75) (end 4.75 3.75) (layer "F.CrtYd") (width 0.05))
+    (fp_line (start -3 -3) (end 0 -3) (layer "F.Fab") (width 0.1))
+    (fp_line (start 0 -3) (end 3 -3) (layer "F.Fab") (width 0.1))
+    (fp_line (start 3 3) (end -3 3) (layer "F.Fab") (width 0.1))
+    (fp_line (start 3 -3) (end 3 3) (layer "F.Fab") (width 0.1))
+    (fp_line (start -3 3) (end -3 -3) (layer "F.Fab") (width 0.1))
+    (fp_circle (center 0 0) (end -2 0.25) (layer "F.Fab") (width 0.1) (fill none))
+    (pad "1" thru_hole circle (at -3.25 -2.25) (size 2 2) (drill 1.1) (layers *.Cu *.Mask)
+      (net 1 "+9V") (pinfunction "1") (pintype "passive"))
+    (pad "2" thru_hole circle (at 3.25 -2.25) (size 2 2) (drill 1.1) (layers *.Cu *.Mask)
+      (net 1 "+9V") (pinfunction "2") (pintype "passive"))
+    (pad "3" thru_hole circle (at -3.25 2.25) (size 2 2) (drill 1.1) (layers *.Cu *.Mask)
+      (net 8 "Net-(BT1-Pad1)") (pinfunction "K") (pintype "passive"))
+    (pad "4" thru_hole circle (at 3.25 2.25) (size 2 2) (drill 1.1) (layers *.Cu *.Mask)
+      (net 8 "Net-(BT1-Pad1)") (pinfunction "A") (pintype "passive"))
+    (model "${KICAD6_3DMODEL_DIR}/Button_Switch_THT.3dshapes/SW_PUSH_6mm.wrl"
+      (offset (xyz -3.25 2.25 0))
+      (scale (xyz 1 1 1))
+      (rotate (xyz 0 0 0))
+    )
+  )
   (footprint "Resistor_THT:R_Axial_DIN0207_L6.3mm_D2.5mm_P7.62mm_Horizontal" (layer "F.Cu")
     (at 113 48.19 -90)
@@
   )
   (gr_rect (start 20 20) (end 120 70) (layer "Edge.Cuts") (width 0.1) (fill none))
-  (segment (start 64 25) (end 70.18 31.18) (width 0.5) (layer "F.Cu") (net 1))
   (segment (start 70.18 31.18) (end 77.8 31.18) (width 0.5) (layer "F.Cu") (net 1))
-  (segment (start 28 25) (end 64 25) (width 0.5) (layer "F.Cu") (net 1))
-  (segment (start 28 25) (end 28 32.19) (width 0.5) (layer "F.Cu") (net 1))
+  (segment (start 63.75 24.75) (end 70.18 31.18) (width 0.5) (layer "F.Cu") (net 1))
+  (segment (start 28.559511 32.749511) (end 28 32.19) (width 0.5) (layer "F.Cu") (net 1))
+  (segment (start 39.25 24.75) (end 63.75 24.75) (width 0.5) (layer "F.Cu") (net 1))
+  (segment (start 37.750489 32.749511) (end 28.559511 32.749511) (width 0.5) (layer "F.Cu") (net 1))
+  (segment (start 39.25 31.25) (end 39.25 24.75) (width 0.5) (layer "F.Cu") (net 1))
+  (segment (start 39.25 31.25) (end 37.750489 32.749511) (width 0.5) (layer "F.Cu") (net 1))
   (segment (start 44.805 54) (end 37.9525 47.1475) (width 0.5) (layer "F.Cu") (net 3))
   (segment (start 70.18 36.26) (end 67.74 36.26) (width 0.5) (layer "F.Cu") (net 3))
@@
   (segment (start 28 39.81) (end 28 47.1) (width 0.5) (layer "F.Cu") (net 6))
   (segment (start 70.18 33.72) (end 75.26 33.72) (width 0.5) (layer "F.Cu") (net 6))
-  (segment (start 28 39.81) (end 34.09 33.72) (width 0.5) (layer "F.Cu") (net 6))
+  (segment (start 28.19 40) (end 28 39.81) (width 0.5) (layer "F.Cu") (net 6))
   (segment (start 75.26 33.72) (end 77.8 36.26) (width 0.5) (layer "F.Cu") (net 6))
-  (segment (start 34.09 33.72) (end 70.18 33.72) (width 0.5) (layer "F.Cu") (net 6))
+  (segment (start 70.18 33.72) (end 65.28 33.72) (width 0.5) (layer "F.Cu") (net 6))
+  (segment (start 59 40) (end 28.19 40) (width 0.5) (layer "F.Cu") (net 6))
   (segment (start 27.9525 47.1475) (end 27.9525 54.6475) (width 0.5) (layer "F.Cu") (net 6))
   (segment (start 28 47.1) (end 27.9525 47.1475) (width 0.5) (layer "F.Cu") (net 6))
   (segment (start 27.9525 54.6475) (end 32.9525 59.6475) (width 0.5) (layer "F.Cu") (net 6))
+  (segment (start 65.28 33.72) (end 59 40) (width 0.5) (layer "F.Cu") (net 6))
+  (segment (start 34.5 25) (end 34.75 24.75) (width 0.5) (layer "F.Cu") (net 8))
+  (segment (start 34.75 24.75) (end 34.75 31.25) (width 0.5) (layer "F.Cu") (net 8))
+  (segment (start 28 25) (end 34.5 25) (width 0.5) (layer "F.Cu") (net 8))
   (zone (net 2) (net_name "GND") (layer "F.Cu") (hatch edge 0.508)
     (connect_pads (clearance 0.508))

Commit message: pcb design for board rev 1
Parts:
- R1: value 50K -> 1K
- RV1: value 50K -> 10K
- U1: footprint timer_footprints:DIP-8_W7.62mm_InvertedDualRow -> Package_DIP:DIP-8_W7.62mm
- moved RV1 33.2 mm to (61.0, 51.1)
- moved R1 30.3 mm to (42.2, 59.0), turned to 0 degrees
- moved C1 16.8 mm to (89.0, 59.0)
- moved U1 7.60 mm to (77.8, 31.2), turned to -90 degrees
- moved BT1 3.00 mm to (31.0, 25.0), turned to 0 degrees
- moved SW1 3.00 mm to (40.0, 28.0)
Connections:
- U1 pad 2: /Discharge -> /Threshold
Routing:
- net /Discharge: track 75.5 -> 48.4 mm
- net /Threshold: track 65.4 -> 43.0 mm
- net +9V: track 59.8 -> 73.0 mm
- net Net-(D1-Pad2): track 36.1 -> 41.5 mm
Other:
- board text added: "+"
- board text added: "-"
- board text added: "1K"
- board text added: "Ausgabe"
- board text added: "Created by: CodingChris - Favo - Kanga Schnupperloeten 2022_01_M_1_Rev_1 das-labor.org"
- board text added: "GND Schwarz"
- board text added: "JLCJLCJLCJLC"
- board text added: "LED"
- board text added: "Rot 9V"
- board text added: "Zeitbestimmende Bauteile"

Commit message: qr code maybe?
Other:
- board text added: "10K"
- board text added: "50uF"
- board text added: "Entladewiderstand RV1"
- board text added: "Gedrückthalten zum Anschalten"
- board text added: "Ladewiderstand R1 + RV1"
- board text added: "Lötworkshop Informationen wiki.das-labor.org/w/Lötworkshops"
- board text added: "NE555 Timer"
- board text added: "Vorwiderstand Strombegrenzung"
- board text added: "τ = R*C"
Changed lines of the file:
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@@
     (property "Sheetname" "")
     (attr through_hole)
-    (fp_text reference "U1" (at 3.81 -2.33 90) (layer "F.SilkS")
+    (fp_text reference "U1" (at 1.8 -2.7 180) (layer "F.SilkS")
       (effects (font (size 1 1) (thickness 0.15)))
     )
@@
     (property "Sheetname" "")
     (attr through_hole)
-    (fp_text reference "RV1" (at -2.1475 -5.0475 180) (layer "F.SilkS")
+    (fp_text reference "RV1" (at -0.6475 -14.5475 180) (layer "F.SilkS")
       (effects (font (size 1 1) (thickness 0.15)))
     )
@@
     (property "Sheetname" "")
     (attr through_hole)
-    (fp_text reference "R1" (at 3.81 -2.37) (layer "F.SilkS")
+    (fp_text reference "R1" (at 1.31 -2.5) (layer "F.SilkS")
       (effects (font (size 1 1) (thickness 0.15)))
     )
@@
     (property "Sheetname" "")
     (attr through_hole)
-    (fp_text reference "C1" (at 1 -3.75) (layer "F.SilkS")
+    (fp_text reference "C1" (at -0.5 -3.75) (layer "F.SilkS")
       (effects (font (size 1 1) (thickness 0.15)))
     )
@@
     (property "Sheetname" "")
     (attr through_hole)
-    (fp_text reference "SW1" (at 0 -4.25 90) (layer "F.SilkS")
+    (fp_text reference "SW1" (at -1.5 -5.5 180) (layer "F.SilkS")
       (effects (font (size 1 1) (thickness 0.15)))
     )
@@
     )
   )
-  (gr_line (start 101 45) (end 20 45) (layer "F.SilkS") (width 0.15))
+  (gr_line (start 101 42) (end 20 42) (layer "F.SilkS") (width 0.15))
   (gr_line (start 101 70) (end 101 20) (layer "F.SilkS") (width 0.15))
+  (gr_line (start 74.5 59) (end 87 59) (layer "F.SilkS") (width 0.15))
+  (gr_line (start 23 59) (end 40.5 59) (layer "F.SilkS") (width 0.15))
+  (gr_line (start 94 59) (end 100 59) (layer "F.SilkS") (width 0.15))
+  (gr_line (start 51.5 59) (end 57.5 59) (layer "F.SilkS") (width 0.15))
   (gr_rect (start 20 20) (end 120 70) (layer "Edge.Cuts") (width 0.1) (fill none))
   (gr_text "Created by: CodingChris - Favo - Kanga\nSchnupperloeten 2022_01_M_1_Rev_1\ndas-labor.org" (at 102 66) (layer "B.SilkS")
     (effects (font (size 1 1) (thickness 0.15)) (justify mirror))
   )
+  (gr_text "Lötworkshop Informationen\nwiki.das-labor.org/w/Lötworkshops" (at 73 66) (layer "B.SilkS")
+    (effects (font (size 1 1) (thickness 0.15)) (justify mirror))
+  )
   (gr_text "JLCJLCJLCJLC" (at 113.5 22) (layer "B.SilkS")
     (effects (font (size 1 1) (thickness 0.15)) (justify mirror))
@@
     (effects (font (size 1 1) (thickness 0.15)))
   )
-  (gr_text "Zeitbestimmende Bauteile" (at 32 46.5) (layer "F.SilkS")
+  (gr_text "Entladewiderstand\nRV1" (at 51 51.5) (layer "F.SilkS")
+    (effects (font (size 1 1) (thickness 0.15)))
+  )
+  (gr_text "Zeitbestimmende Bauteile" (at 31.5 43) (layer "F.SilkS")
+    (effects (font (size 1 1) (thickness 0.15)))
+  )
+  (gr_text "1K" (at 43.5 61.5) (layer "F.SilkS")
     (effects (font (size 1 1) (thickness 0.15)))
   )
@@
     (effects (font (size 1 1) (thickness 0.15)))
   )
+  (gr_text "Gedrückthalten zum Anschalten" (at 41 34) (layer "F.SilkS")
+    (effects (font (size 1 1) (thickness 0.15)))
+  )
+  (gr_text "Ladewiderstand\nR1 + RV1" (at 51 48) (layer "F.SilkS")
+    (effects (font (size 1 1) (thickness 0.15)))
+  )
+  (gr_text "50uF" (at 89 62.5) (layer "F.SilkS")
+    (effects (font (size 1 1) (thickness 0.15)))
+  )
   (gr_text "Ausgabe" (at 105 22.5) (layer "F.SilkS")
     (effects (font (size 1 1) (thickness 0.15)))
   )
+  (gr_text "Vorwiderstand\nStrombegrenzung" (at 108 45) (layer "F.SilkS")
+    (effects (font (size 1 1) (thickness 0.15)))
+  )
+  (gr_text "10K" (at 75.5 52) (layer "F.SilkS")
+    (effects (font (size 1 1) (thickness 0.15)))
+  )
+  (gr_text "τ = R*C" (at 25 44.5) (layer "F.SilkS")
+    (effects (font (size 1 1) (thickness 0.15)))
+  )
   (gr_text "1K" (at 110 51) (layer "F.SilkS")
     (effects (font (size 1 1) (thickness 0.15)))
   )
+  (gr_text "NE555\nTimer" (at 82 35.5) (layer "F.SilkS")
+    (effects (font (size 1 1) (thickness 0.15)))
+  )
